Commit message: master

File: urdf/megarover3.gazebo.xacro (robot description, xacro)
@@ -1,4 +1,4 @@
 <?xml version="1.0"?>
-<robot name="megarover3_sim" xmlns:xacro="http://ros.org/wiki/xacro">
+<robot name="megarover3" xmlns:xacro="http://ros.org/wiki/xacro">
   <xacro:arg name="laser_visual"  default="false"/>
   <xacro:arg name="camera_visual" default="false"/>
@@ -13,21 +13,37 @@
       <xacro:property name="imu_frame" value="$(arg tf_prefix)/imu_link" />
   </xacro:unless>
+  <gazebo reference="camera_stay_link">
+    <material>Gazebo/Grey</material>
+  </gazebo>
+  <xacro:property name="body_color" value="Gazebo/Silver" />
+  <xacro:property name="wheel_color" value="Gazebo/DarkGrey" />
   <gazebo reference="base_link">
-    <selfCollide>false</selfCollide>
-    <mu1 value="0.0" />
-    <mu2 value="0.0" />
+    <material>${body_color}</material>
+    <mu1>0.1</mu1>
+    <mu2>0.1</mu2>
+    <kp>1e6</kp>
+    <kd>100.0</kd>
+    <minDepth>0.001</minDepth>
+    <maxVel>1.0</maxVel>
+  </gazebo>
+  <gazebo reference="wheel_right_link">
+    <mu1>1.0</mu1>
+    <mu2>1.0</mu2>
+    <fdir1>1 0 0</fdir1>
+    <kp>1e6</kp>
+    <kd>10.0</kd>
+    <minDepth>0.0001</minDepth>
+    <maxVel>0.1</maxVel>
+    <material>${wheel_color}</material>
   </gazebo>
   <gazebo reference="wheel_left_link">
-    <selfCollide>false</selfCollide>
-    <mu1 value="1.0" />
-    <mu2 value="1.0" />
-  </gazebo>
-  <gazebo reference="wheel_right_link">
-    <selfCollide>false</selfCollide>
-    <mu1 value="1.0" />
-    <mu2 value="1.0" />
-  </gazebo>
-  <gazebo reference="camera_stay_link">
-    <material>Gazebo/Grey</material>
+    <mu1>1.0</mu1>
+    <mu2>1.0</mu2>
+    <fdir1>1 0 0</fdir1>
+    <kp>1e6</kp>
+    <kd>10.0</kd>
+    <minDepth>0.0001</minDepth>
+    <maxVel>0.1</maxVel>
+    <material>${wheel_color}</material>
   </gazebo>
   <gazebo>
@@ -41,15 +57,18 @@
       <publishWheelTF>true</publishWheelTF>
       <publishTf>true</publishTf>
-      <publishWheelJointState>true</publishWheelJointState>
+      <publishWheelJointState>false</publishWheelJointState>
       <legacyMode>false</legacyMode>
       <updateRate>30</updateRate>
       <leftJoint>wheel_left_joint</leftJoint>
       <rightJoint>wheel_right_joint</rightJoint>
-      <wheelSeparation>0.284</wheelSeparation>
-      <wheelDiameter>0.152</wheelDiameter>
-      <!-- <wheelAcceleration>1</wheelAcceleration> -->
-      <!-- <wheelTorque>10</wheelTorque> -->
+      <wheelSeparation>0.272</wheelSeparation>
+      <wheelDiameter>0.140</wheelDiameter>
+      <wheelAcceleration>1.0</wheelAcceleration>
+      <wheelTorque>30</wheelTorque>
       <rosDebugLevel>na</rosDebugLevel>
     </plugin>
+  </gazebo>
+  <gazebo>
+    <plugin name="gazebo_ros_control" filename="libgazebo_ros_control.so" />
   </gazebo>
   <gazebo reference="base_scan">

File: urdf/megarover3_mesh.urdf.xacro (robot description, xacro)
@@ -2,36 +2,14 @@
 <robot name="megarover3" xmlns:xacro="http://ros.org/wiki/xacro">
   <xacro:include filename="$(find megarover_samples)/urdf/common.xacro"/>
-  <!-- <xacro:include filename="$(find turtlebot3_description)/urdf/common_properties.xacro"/> -->
+  <xacro:include filename="$(find turtlebot3_description)/urdf/common_properties.xacro"/>
   <xacro:include filename="$(find potbot_example)/urdf/megarover3.gazebo.xacro"/>
-  <xacro:include filename="$(find megarover_description)/urdf/materials.xacro" />
-  <xacro:include filename="$(find megarover_description)/urdf/mega3.gazebo" />
-  <!-- OPTION: LRF TG30 -->
-  <!-- <xacro:include filename="$(find vs_rover_options_description)/urdf/lrf/tg30_mega3.xacro" /> -->
-  <!-- OPTION: bumper sensor -->
-  <xacro:include filename="$(find vs_rover_options_description)/urdf/bumper/bumper_mega3.xacro" />
-  <xacro:bumperbaseboard prefix="front" parent="base_link" xyz="0 0.19 0.02" z_dir="180" />
-  <xacro:bumperbaseboard prefix="back" parent="base_link" xyz="0 -0.19 0.02" z_dir="0" />
-  <!-- OPTION: camera stay -->
-  <!-- <xacro:include filename="$(find vs_rover_options_description)/urdf/cam_stay/cam_stay_mega3.xacro" /> -->
-  <!-- OPTION: Intel Realsense depth camera D435i (camera stay required) -->
-  <!-- <xacro:include filename="$(find vs_rover_options_description)/urdf/depth_cam/_d435i.urdf.xacro" />
-  <xacro:sensor_d435i parent="cam_mount_link" use_nominal_extrinsics="true">
-    <origin xyz="0.0295 0 0.0095" rpy="0 0 0" />
-  </xacro:sensor_d435i> -->
-  <!-- OPTION: AMIR 740 (disabled by default because of interference with camera stay)-->
-  <!-- <xacro:include filename="$(find amir_description)/urdf/amir_for_rover.xacro" />
-  <joint name="base_fixed" type="fixed">
-    <origin xyz="0.0 0.03 0.398" rpy="0 0 0" />
-    <parent link="base_link" />
-    <child link="link0_1" />
-  </joint> -->
   <xacro:property name="wheel_radius" value="0.076"/>
   <xacro:property name="wheel_length" value="0.03"/>
   <xacro:property name="wheel_mass" value="0.823"/>
-  <link name="base_footprint" />
+  <link name="base_footprint"/>
   <joint name="base_joint" type="fixed">
-    <parent link="base_footprint" />
+    <parent link="base_footprint"/>
     <child link="base_link" />
-    <origin xyz="-0.1 0 0" rpy="0 0 -${M_PI/2}" />
+    <origin xyz="-0.1 0 0" rpy="0 0 -1.5708" />
   </joint>
   <link name="base_link">
@@ -73,5 +51,5 @@
     <parent link="base_link" />
     <child link="wheel_left_link" />
-    <axis xyz="0.0 0.0 1.0" />
+    <axis xyz="0 0 1" />
   </joint>
   <link name="wheel_left_link">
@@ -107,5 +85,5 @@
     <parent link="base_link" />
     <child link="wheel_right_link" />
-    <axis xyz="0.0 0.0 1.0" />
+    <axis xyz="0 0 1" />
   </joint>
   <link name="wheel_right_link">
@@ -140,5 +118,5 @@
     <parent link="base_link" />
     <child link="base_scan" />
-    <origin xyz="0 0.09 0.223" rpy="0 0 ${M_PI/2}"/>
+    <origin xyz="0 0.18 0.223" rpy="0 0 1.57"/>
   </joint>
   <!-- <link name="base_scan">
@@ -170,5 +148,5 @@
   </link>
   <joint name="camera_stay_joint" type="fixed">
-    <origin xyz="0 0.06 0.305" rpy="0 0 ${M_PI/2}"/>
+    <origin xyz="0 0.15 0.305" rpy="0 0 1.57"/>
     <parent link="base_link"/>
     <child link="camera_stay_link"/>
@@ -196,7 +174,7 @@
   <link name="camera_link">
     <visual>
-      <origin xyz="0 0 0" rpy="${M_PI/2} 0 ${M_PI/2}"/>
-      <geometry>
-        <mesh filename="package://vs_rover_options_description/meshes/depth_cam/d435.dae" />
+      <origin xyz="0 0 0" rpy="0 0 0"/>
+      <geometry>
+        <box size="0.03 0.165 0.03"/>
       </geometry>
       <material name="white" />
@@ -206,4 +184,5 @@
     <parent link="camera_link"/>
     <child link="imu_link"/>
+    <!-- <origin xyz="0 0 0" rpy="3.14 0 0"/> -->
     <origin xyz="0 0 0" rpy="0 1.57 0"/>
   </joint>
